File: schematics/KiCad/Z80ATmega128.kicad_sch (KiCad schematic)
At the start: 68 parts, among them J1 AVR-ISP-6, J2 DC 5V, J3 DC 5V, J4 Z80[1..20], J5 Z80[21..40], SW1 Power, U1 74HC125, U10 74HC08, U11 74HC32, U12 74HC32, U13 74LS08, U14 74HC74, U2 74HC04, U3 74AC573, U4 74HCT574, U5 AE-CH340E-TYPEC, U6 74HC125, U7 74HC244, U8 74HCT245, U9 AE-CH340E-TYPEC, Y1 16MHz, Y2 8MHz

Commit message: Fixed bug of WAIT generator circuit
Clock circuit is moved to 2nd layer.
Parts:
- removed C10, C11: 22p, Capacitor_THT:C_Disc_D3.8mm_W2.6mm_P2.50mm, symbol Device:C
- removed R15: 1M, Resistor_THT:R_Axial_DIN0204_L3.6mm_D1.6mm_P7.62mm_Horizontal, symbol Device:R
- removed R16: 100, Resistor_THT:R_Axial_DIN0204_L3.6mm_D1.6mm_P7.62mm_Horizontal, symbol Device:R
- removed TP3: 4MHz, TestPoint:TestPoint_Loop_D2.50mm_Drill1.0mm, symbol Connector:TestPoint
- removed unit 1 of U14
- removed unit 4 of U2
- removed unit 5 of U2
- removed Y2: 8MHz, Crystal:Crystal_HC18-U_Vertical, symbol Device:Crystal
- added C18: 0.1u, Capacitor_THT:C_Disc_D3.8mm_W2.6mm_P2.50mm, symbol Device:C
- added U14: 74LS32, symbol 74xx:74LS32
- renumbered C12 to C10, C13 to C11, C14 to C12, C15 to C13, C16 to C14, C17 to C15, C18 to C16, C19 to C17, U14 to U15
Connections:
- net GND: now also C18.2, U14.1, U14.12, U14.13, U14.2, U14.4, U14.5, U14.7 (GND)
- net VCC: now also C18.1, U14.14 (VCC)
- net /IORQ: now also U14.10
- net /WAIT: now also U14.8; no longer U10.1, U15.9 (Q)
- new net: U10.1, U14.9, U15.9 (Q)
- no-connect marks 15 -> 18
Other:
- sheet Reset ports: added 4MHz; removed /ST
- moved on the sheet: C17, U10A, U12C, U13D, U13E, U15B
