File: schematics/KiCad/Z80ATmega128.kicad_sch (KiCad schematic)
At the start: 61 parts, among them J1 AVR-ISP-6, J2 Z80[1..20], J3 DC 5V, J4 Z80[21..40], J5 DC 5V, SW1 Power, U1 74HC125, U10 74HC32, U11 74HC32, U12 74HC74, U13 74HC32, U2 74AC573, U3 74HCT574, U4 74HC04, U5 74HC125, U6 74HC244, U7 74HCT245, U8 74HC08, U9 74HC08, Y1 16MHz

Commit message: Update schematics
Parts:
- added C3: 0.1u, Capacitor_THT:C_Disc_D3.8mm_W2.6mm_P2.50mm, symbol Device:C
- C10: renamed from C9; footprint Capacitor_THT:CP_Radial_Tantal_D5.0mm_P2.50mm -> Capacitor_THT:CP_Radial_D5.0mm_P2.50mm
- renumbered C10 to C11, C11 to C12, C12 to C13, C13 to C14, C14 to C15, C15 to C16, C16 to C17, C17 to C18, C18 to C19, C3 to C4, C4 to C5, C5 to C6, C6 to C7, C7 to C8, C8 to C9, U5 to U1, U11 to U10, U9 to U11, U8 to U11, U6 to U5, U7 to U6, U9 to U7, U8 to U7, U1 to U8, U5 to U8, U10 to U9
Connections:
- net /BACK is gone; now on net /BUSACK: CPU1.23 (~{BUSACK}), R11.2, U7.12
- net GND: now also C11.1, C12.1, C13.1, C14.1, C15.1, C16.1, C17.1, C18.1, C19.1, C2.2, C3.1; no longer C11.2, C12.2, C13.2, C14.2, C15.2, C16.2, C17.2, C18.2, C19.2, C2.1
- net Reset//Z80_SWRST: now also R3.1; no longer R3.2
- net VCC: now also C11.2, C12.2, C13.2, C14.2, C15.2, C16.2, C17.2, C18.2, C19.2, C2.1, R12.2, R3.2, C3.2; no longer C11.1, C12.1, C13.1, C14.1, C15.1, C16.1, C17.1, C18.1, C19.1, C2.2, R12.1, R3.1
- net /BUSACK: no longer CPU2.32 (PD7), U1.10, U2.1 (OE), U4.1, U5.1 (1OE), U5.19 (2OE), U7.11, U8.13
- net /BUSRQ: no longer J4.16 (Pin_16)
- net /Z80_BUSRQ: now reaches CPU1.25 (~{BUSRQ}), JP1.2 (C)
- net /Z80_BUSRQ: now also J4.16 (Pin_16), R12.1; no longer R12.2
- net at Y1.1: now also CPU2.23 (XTAL2); no longer CPU2.24 (XTAL1)
- net at Y1.3: now also CPU2.24 (XTAL1); no longer CPU2.23 (XTAL2)
- new net: CPU2.32 (PD7), U1.10, U2.1 (OE), U4.1, U5.1 (1OE), U5.19 (2OE), U7.11, U8.13
Other:
- moved on the sheet: C2

Commit message: Swap R4 and R5, Change min_resolved_spokes 2 to 1.
Connections:
- net /NMI: now also R4.2; no longer R5.2
- net /XINT: now also R5.2; no longer R4.2
Other:
- moved on the sheet: R4, R5
Changed lines of the file:
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@@
     )
   )
-  (symbol (lib_id "Device:R") (at 383.54 53.34 0) (unit 1)
-    (in_bom yes) (on_board yes) (dnp no)
-    (property "Reference" "R5" (at 383.54 44.45 90)
-      (effects (font (size 1.27 1.27)))
-    )
-    (property "Value" "10K" (at 383.54 40.64 90)
-      (effects (font (size 1.27 1.27)))
-    )
-    (property "Footprint" "Resistor_THT:R_Axial_DIN0204_L3.6mm_D1.6mm_P7.62mm_Horizontal" (at 381.762 53.34 90)
-      (effects (font (size 1.27 1.27)) hide)
-    )
-    (property "Datasheet" "~" (at 383.54 53.34 0)
+  (symbol (lib_id "Device:R") (at 381 53.34 0) (unit 1)
+    (in_bom yes) (on_board yes) (dnp no)
+    (property "Reference" "R5" (at 381 44.45 90)
+      (effects (font (size 1.27 1.27)))
+    )
+    (property "Value" "10K" (at 381 40.64 90)
+      (effects (font (size 1.27 1.27)))
+    )
+    (property "Footprint" "Resistor_THT:R_Axial_DIN0204_L3.6mm_D1.6mm_P7.62mm_Horizontal" (at 379.222 53.34 90)
+      (effects (font (size 1.27 1.27)) hide)
+    )
+    (property "Datasheet" "~" (at 381 53.34 0)
       (effects (font (size 1.27 1.27)) hide)
     )
@@
     )
   )
-  (symbol (lib_id "Device:R") (at 381 53.34 0) (unit 1)
-    (in_bom yes) (on_board yes) (dnp no)
-    (property "Reference" "R4" (at 381 44.45 90)
-      (effects (font (size 1.27 1.27)))
-    )
-    (property "Value" "10K" (at 381 40.64 90)
-      (effects (font (size 1.27 1.27)))
-    )
-    (property "Footprint" "Resistor_THT:R_Axial_DIN0204_L3.6mm_D1.6mm_P7.62mm_Horizontal" (at 379.222 53.34 90)
-      (effects (font (size 1.27 1.27)) hide)
-    )
-    (property "Datasheet" "~" (at 381 53.34 0)
-      (effects (font (size 1.27 1.27)) hide)
-    )
+  (symbol (lib_id "Device:R") (at 383.54 53.34 0) (unit 1)
+    (in_bom yes) (on_board yes) (dnp no)
+    (property "Reference" "R4" (at 383.54 44.45 90)
+      (effects (font (size 1.27 1.27)))
+    )
+    (property "Value" "10K" (at 383.54 40.64 90)
+      (effects (font (size 1.27 1.27)))
+    )
+    (property "Footprint" "Resistor_THT:R_Axial_DIN0204_L3.6mm_D1.6mm_P7.62mm_Horizontal" (at 381.762 53.34 90)
+      (effects (font (size 1.27 1.27)) hide)
+    )
+    (property "Datasheet" "~" (at 383.54 53.34 0)
+      (effects (font (size 1.27 1.27)) hide)
+    )

Commit message: Update for PCB design
Parts:
- CPU2: symbol MCU_Microchip_ATmega:ATmega128-16A -> 46nori_Library:ATmega128-16A
Connections:
- net 4MHz: now also U7.10; no longer U11.2
- net /INT0: now also U11.1; no longer U7.9
- net /INT4: now also U11.2; no longer U7.10
- net /WAIT_0: now also U7.9; no longer U11.1
- net at U12.11 (C): now also U7.8; no longer U11.3
- net at U3.1 (OE): now also U11.3; no longer U7.8
Other:
- moved on the sheet: U11A, U7C
Changed lines of the file:
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@@
   (junction (at 340.36 156.21) (diameter 0) (color 0 0 0 0)
   )
+  (junction (at 372.11 187.96) (diameter 0) (color 0 0 0 0)
+  )
   (junction (at 54.61 227.33) (diameter 0) (color 0 0 0 0)
   )
@@
   (junction (at 50.8 49.53) (diameter 0) (color 0 0 0 0)
   )
-  (junction (at 372.11 187.96) (diameter 0) (color 0 0 0 0)
-  )
   (junction (at 38.1 227.33) (diameter 0) (color 0 0 0 0)
   )
@@
     )
   )
-  (symbol (lib_id "74xx:74LS08") (at 344.17 241.3 0) (mirror y) (unit 1)
+  (symbol (lib_id "74xx:74LS08") (at 364.49 185.42 0) (mirror y) (unit 1)
     (in_bom yes) (on_board yes) (dnp no)
-    (property "Reference" "U11" (at 328.93 240.03 0)
+    (property "Reference" "U11" (at 361.95 177.8 0)
       (effects (font (size 1.27 1.27)))
     )
-    (property "Value" "74HC08" (at 330.2 242.57 0)
+    (property "Value" "74HC08" (at 363.22 180.34 0)
       (effects (font (size 1.27 1.27)))
     )
-    (property "Footprint" "Package_DIP:DIP-14_W7.62mm_Socket" (at 344.17 241.3 0)
+    (property "Footprint" "Package_DIP:DIP-14_W7.62mm_Socket" (at 364.49 185.42 0)
       (effects (font (size 1.27 1.27)) hide)
     )
-    (property "Datasheet" "http://www.ti.com/lit/gpn/sn74LS08" (at 344.17 241.3 0)
+    (property "Datasheet" "http://www.ti.com/lit/gpn/sn74LS08" (at 364.49 185.42 0)
       (effects (font (size 1.27 1.27)) hide)
     )
@@
     )
   )
-  (symbol (lib_id "MCU_Microchip_ATmega:ATmega128-16A") (at 120.65 88.9 0) (unit 1)
+  (symbol (lib_id "46nori_Library:ATmega128-16A") (at 120.65 88.9 0) (unit 1)
     (in_bom yes) (on_board yes) (dnp no)
     (property "Reference" "CPU2" (at 128.27 139.7 0)
@@
     )
   )
-  (symbol (lib_id "74xx:74LS08") (at 364.49 185.42 0) (mirror y) (unit 3)
-    (in_bom yes) (on_board yes) (dnp no) (fields_autoplaced)
-    (property "Reference" "U7" (at 364.49 176.53 0)
+  (symbol (lib_id "74xx:74LS08") (at 344.17 241.3 0) (mirror y) (unit 3)
+    (in_bom yes) (on_board yes) (dnp no)
+    (property "Reference" "U7" (at 334.01 238.76 0)
       (effects (font (size 1.27 1.27)))
     )
-    (property "Value" "74HC08" (at 364.49 179.07 0)
+    (property "Value" "74HC08" (at 335.28 243.84 0)
       (effects (font (size 1.27 1.27)))
     )
-    (property "Footprint" "Package_DIP:DIP-14_W7.62mm_Socket" (at 364.49 185.42 0)
+    (property "Footprint" "Package_DIP:DIP-14_W7.62mm_Socket" (at 344.17 241.3 0)
       (effects (font (size 1.27 1.27)) hide)
     )
-    (property "Datasheet" "http://www.ti.com/lit/gpn/sn74LS08" (at 364.49 185.42 0)
+    (property "Datasheet" "http://www.ti.com/lit/gpn/sn74LS08" (at 344.17 241.3 0)
       (effects (font (size 1.27 1.27)) hide)
     )
