File: schematics/KiCad/Z80ATmega128.kicad_sch (KiCad schematic)
At the start: 62 parts, among them J1 AVR-ISP-6, J2 Z80[1..20], J3 DC 5V, J4 Z80[21..40], J5 DC 5V, SW1 Power, U1 74HC125, U10 74HC32, U11 74HC08, U12 74HC74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

Commit message: Update document and BOM of schematics.
Parts:
- C1, C11, C12, C13, C14, C15, C16, C17, C18, C19, C2, C3, C4, C5, C6, C7, C8, C9: 部品名 (none) -> 0.1uF/50V 積層セラミックコンデンサ
- C10: 部品名 (none) -> 100uF/25V 電解コンデンサ
- CPU1: 部品名 (none) -> Z80A CPU (NMOS)
- CPU2: 部品名 (none) -> ATmega128-16A
- D1: 部品名 (none) -> LED (緑)
- J1: 購入先(参考) (none) -> https://akizukidenshi.com/catalog/g/gC-13175/; 部品名 (none) -> ボックスヘッダ 2x3
- J2, J4: 購入先(参考) (none) -> https://akizukidenshi.com/catalog/g/gC-00167/; 部品名 (none) -> ピンヘッダ 1x20
- J3: 購入先(参考) (none) -> https://akizukidenshi.com/catalog/g/gP-01306/; 部品名 (none) -> ターミナルブロック
- J5: 購入先(参考) (none) -> https://akizukidenshi.com/catalog/g/gC-06568/; 部品名 (none) -> 2.1mm標準DCジャック
- JP1, JP2: 部品名 (none) -> ピンヘッダ 1x3
- R1, R10, R11, R12, R13, R14, R2, R3, R4, R5, R6, R7, R8, R9: 部品名 (none) -> 1/4Wカーボン抵抗
- SRAM1, SRAM2: 部品名 (none) -> 256KBit SRAM
- SW1: 購入先(参考) (none) -> https://akizukidenshi.com/catalog/g/gP-00301/; 部品名 (none) -> トグルスイッチ 2回路2接点
- TP1: 購入先(参考) (none) -> https://akizukidenshi.com/catalog/g/gP-07588/; 部品名 (none) -> チェック端子(赤)
- TP2: 購入先(参考) (none) -> https://akizukidenshi.com/catalog/g/gP-07591/; 部品名 (none) -> チェック端子(黒)
- U1, U8: 部品名 (none) -> 74HC125
- U10, U13, U9: 部品名 (none) -> 74HC32
- U11, U7: 部品名 (none) -> 74HC08
- U12: 部品名 (none) -> 74HC74
- U2: 部品名 (none) -> 74AC573
- U3: 部品名 (none) -> 74HCT574
- U4: 部品名 (none) -> 74HC04
- U5: 部品名 (none) -> 74HC244
- U6: 部品名 (none) -> 74HCT245
- Y1: 購入先(参考) (none) -> https://akizukidenshi.com/catalog/g/gP-09576/; 部品名 (none) -> 16MHz セラミック発振子

Commit message: Update schematics and document.
Parts:
- J1: footprint Connector_PinHeader_2.54mm:PinHeader_2x03_P2.54mm_Vertical -> 46nori:BoxHeader_2x03_2.54mm
- SW1: footprint Button_Switch_THT:SW_CuK_JS202011CQN_DPDT_Straight -> 46nori:2MD1-T1-B4-VS2-Q-E; symbol Switch:SW_Push_DPDT -> 46nori_Library:SW_Toggle_2x2
Connections:
- net ExtIO/+5V: now also SW1.5 (B); no longer SW1.2 (B)
- net VCC: now also SW1.1 (A), SW1.4 (A); no longer SW1.3 (C), SW1.6 (C)
- net /RD: no longer CPU2.34 (PG1), U7.2, U8.12
- net /WR: no longer CPU2.33 (PG0), U1.9, U7.1
- net at JP2.2 (C): now also SW1.2 (B); no longer SW1.5 (B)
- net ALE renamed AVR_ALE
- new net /AVR_RD: CPU2.34 (PG1), U7.2, U8.12
- new net /AVR_WR: CPU2.33 (PG0), U1.9, U7.1
Changed lines of the file:
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@@
   (junction (at 365.76 87.63) (diameter 0) (color 0 0 0 0)
   )
+  (junction (at 54.61 204.47) (diameter 0) (color 0 0 0 0)
+  )
   (junction (at 63.5 99.06) (diameter 0) (color 0 0 0 0)
   )
@@
   (junction (at 50.8 49.53) (diameter 0) (color 0 0 0 0)
   )
+  (junction (at 54.61 214.63) (diameter 0) (color 0 0 0 0)
+  )
   (junction (at 38.1 227.33) (diameter 0) (color 0 0 0 0)
   )
@@
   (junction (at 31.75 276.86) (diameter 0) (color 0 0 0 0)
   )
-  (junction (at 54.61 204.47) (diameter 0) (color 0 0 0 0)
-  )
   (junction (at 278.13 38.1) (diameter 0) (color 0 0 0 0)
   )
@@
   (junction (at 378.46 85.09) (diameter 0) (color 0 0 0 0)
   )
-  (junction (at 54.61 214.63) (diameter 0) (color 0 0 0 0)
-  )
   (junction (at 375.92 74.93) (diameter 0) (color 0 0 0 0)
   )
@@
     (stroke (width 0) (type default))
   )
+  (wire (pts (xy 54.61 204.47) (xy 54.61 214.63))
+    (stroke (width 0) (type default))
+  )
   (bus (pts (xy 251.46 58.42) (xy 251.46 60.96))
     (stroke (width 0) (type default))
@@
     (stroke (width 0) (type default))
   )
-  (wire (pts (xy 54.61 214.63) (xy 54.61 217.17))
-    (stroke (width 0) (type default))
-  )
   (wire (pts (xy 306.07 44.45) (xy 314.96 44.45))
     (stroke (width 0) (type default))
@@
     (stroke (width 0) (type default))
   )
-  (wire (pts (xy 54.61 204.47) (xy 54.61 214.63))
-    (stroke (width 0) (type default))
-  )
   (wire (pts (xy 68.58 134.62) (xy 76.2 134.62))
     (stroke (width 0) (type default))
@@
     (stroke (width 0) (type default))
   )
+  (wire (pts (xy 54.61 214.63) (xy 54.61 217.17))
+    (stroke (width 0) (type default))
+  )
   (wire (pts (xy 229.87 166.37) (xy 229.87 177.8))
     (stroke (width 0) (type default))
@@
     (effects (font (size 1.27 1.27)) (justify left bottom))
   )
-  (label "{slash}WR" (at 95.25 71.12 0) (fields_autoplaced)
+  (label "{slash}AVR_WR" (at 95.25 71.12 0) (fields_autoplaced)
     (effects (font (size 1.27 1.27)) (justify left bottom))
   )
@@
     (effects (font (size 1.27 1.27)) (justify right bottom))
   )
-  (label "{slash}RD" (at 95.25 73.66 0) (fields_autoplaced)
+  (label "{slash}AVR_RD" (at 95.25 73.66 0) (fields_autoplaced)
     (effects (font (size 1.27 1.27)) (justify left bottom))
   )
@@
     (effects (font (size 1.27 1.27)) (justify left bottom))
   )
-  (label "ALE" (at 96.52 76.2 0) (fields_autoplaced)
+  (label "AVR_ALE" (at 96.52 76.2 0) (fields_autoplaced)
     (effects (font (size 1.27 1.27)) (justify left bottom))
   )
@@
       (effects (font (size 1.27 1.27)) (justify right))
     )
-    (property "Footprint" "Connector_PinHeader_2.54mm:PinHeader_2x03_P2.54mm_Vertical" (at 26.67 64.77 90)
+    (property "Footprint" "46nori:BoxHeader_2x03_2.54mm" (at 26.67 64.77 90)
       (effects (font (size 1.27 1.27)) hide)
     )
@@
     )
   )
-  (symbol (lib_id "Switch:SW_Push_DPDT") (at 45.72 207.01 0) (unit 1)
-    (in_bom yes) (on_board yes) (dnp no) (fields_autoplaced)
-    (property "Reference" "SW1" (at 45.72 195.58 0)
+  (symbol (lib_id "46nori_Library:SW_Toggle_2x2") (at 45.72 217.17 0) (mirror x) (unit 1)
+    (in_bom yes) (on_board yes) (dnp no)
+    (property "Reference" "SW1" (at 45.72 193.04 0)
       (effects (font (size 1.27 1.27)))
     )
-    (property "Value" "Power" (at 45.72 198.12 0)
+    (property "Value" "Power" (at 45.72 195.58 0)
       (effects (font (size 1.27 1.27)))
     )
-    (property "Footprint" "Button_Switch_THT:SW_CuK_JS202011CQN_DPDT_Straight" (at 45.72 201.93 0)
+    (property "Footprint" "46nori:2MD1-T1-B4-VS2-Q-E" (at 45.72 217.17 0)
       (effects (font (size 1.27 1.27)) hide)
     )
-    (property "Datasheet" "https://akizukidenshi.com/download/2MD1T2B4M2QN.pdf" (at 45.72 201.93 0)
+    (property "Datasheet" "https://akizukidenshi.com/download/2MD1T2B4M2QN.pdf" (at 45.72 217.17 0)
       (effects (font (size 1.27 1.27)) hide)
     )
-    (property "購入先(参考)" "https://akizukidenshi.com/catalog/g/gP-00301/" (at 45.72 207.01 0)
+    (property "購入先(参考)" "https://akizukidenshi.com/catalog/g/gP-00301/" (at 45.72 217.17 0)
       (effects (font (size 1.27 1.27)) hide)
     )
-    (property "部品名" "トグルスイッチ 2回路2接点" (at 45.72 207.01 0)
+    (property "部品名" "トグルスイッチ 2回路2接点" (at 45.72 217.17 0)
       (effects (font (size 1.27 1.27)) hide)
     )
@@
     (pin "5")
     (pin "6")
+    (pin "7")
+    (pin "8")
     (instances
       (project "Z80ATmega128"
