File: schematics/KiCad/ExtIO_sch.kicad_sch (KiCad schematic)
At the start: 20 parts, among them SW2 SW_DIP_x04, U1 74HC125, U10 AE-CH340E-TYPEC, U14 74HC32, U2 74HC04, U5 AE-CH340E-TYPEC

Commit message: Update schematics
Parts:
- U?: renamed from U10; value AE-CH340E-TYPEC -> AE-CH340E-TYPECH (CH1)
- U?: renamed from U5; value AE-CH340E-TYPEC -> AE-CH340E-TYPEC (CH0)
- renumbered D1 to D?, R2 to R?, R17 to R?, R16 to R?, R13 to R?, R15 to R?, SW2 to SW?, U1 to U?, U2 to U?, U14 to U?
Connections:
- net VCC: now also R?.1; no longer R?.2
- net at D?.2 (A): now also R?.2; no longer R?.1
Other:
- moved on the sheet: R?

Commit message: Update for PCB design
Parts:
- U? (x2): footprint Connector_PinHeader_2.54mm:PinHeader_1x06_P2.54mm_Vertical -> 46nori:AE-CH340E-TYPECH
Changed lines of the file:
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@@
     )
   )
-  (symbol (lib_id "46nori_Library:AE-CH340E-TYPEC") (at 105.41 73.66 0) (unit 1)
+  (symbol (lib_name "AE-CH340E-TYPEC_1") (lib_id "46nori_Library:AE-CH340E-TYPEC") (at 105.41 73.66 0) (unit 1)
     (in_bom yes) (on_board yes) (dnp no) (fields_autoplaced)
     (property "Reference" "U?" (at 104.775 69.85 0)
@@
       (effects (font (size 1.27 1.27)))
     )
-    (property "Footprint" "Connector_PinHeader_2.54mm:PinHeader_1x06_P2.54mm_Vertical" (at 105.41 73.66 0)
+    (property "Footprint" "46nori:AE-CH340E-TYPECH" (at 105.41 73.66 0)
       (effects (font (size 1.27 1.27)) hide)
     )
@@
     )
     (pin "1")
+    (pin "10")
     (pin "2")
     (pin "3")
@@
     (pin "5")
     (pin "6")
+    (pin "7")
+    (pin "8")
+    (pin "9")
     (instances
       (project "Z80ATmega128"
@@
     )
   )
-  (symbol (lib_name "AE-CH340E-TYPEC_1") (lib_id "46nori_Library:AE-CH340E-TYPEC") (at 105.41 25.4 0) (unit 1)
+  (symbol (lib_id "46nori_Library:AE-CH340E-TYPEC") (at 105.41 25.4 0) (unit 1)
     (in_bom yes) (on_board yes) (dnp no) (fields_autoplaced)
     (property "Reference" "U?" (at 104.775 21.59 0)
@@
       (effects (font (size 1.27 1.27)))
     )
-    (property "Footprint" "Connector_PinHeader_2.54mm:PinHeader_1x06_P2.54mm_Vertical" (at 105.41 25.4 0)
+    (property "Footprint" "46nori:AE-CH340E-TYPECH" (at 105.41 25.4 0)
       (effects (font (size 1.27 1.27)) hide)
     )
@@
     )
     (pin "1")
+    (pin "10")
     (pin "2")
     (pin "3")
@@
     (pin "5")
     (pin "6")
+    (pin "7")
+    (pin "8")
+    (pin "9")
     (instances
       (project "Z80ATmega128"

Commit message: Update document and BOM of schematics.
Parts:
- D? (x3): 部品名 (none) -> LED (赤)
- D?: 部品名 (none) -> LED (黄)
- D?: 部品名 (none) -> LED (青)
- R? (x9): 部品名 (none) -> 1/4Wカーボン抵抗
- SW?: 購入先(参考) (none) -> https://akizukidenshi.com/catalog/g/gP-00586/; 部品名 (none) -> 4連DIPスイッチ
- U?: 部品名 (none) -> 74HC125
- U?: value AE-CH340E-TYPECH (CH1) -> AE-CH340E-TYPEC; 購入先(参考) (none) -> https://akizukidenshi.com/catalog/g/gK-14745/; 部品名 (none) -> USB-Cシリアル変換モジュール
- U?: value AE-CH340E-TYPEC (CH0) -> AE-CH340E-TYPEC; 購入先(参考) (none) -> https://akizukidenshi.com/catalog/g/gK-14745/; 部品名 (none) -> USB-Cシリアル変換モジュール
- U?: 部品名 (none) -> 74HC04
- U? (x3): 部品名 (none) -> 74HC32
Changed lines of the file:
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@@
+      (effects (font (size 1.27 1.27)) hide)
+    )
+    (property "購入先(参考)" "" (at 193.04 67.31 0)
+      (effects (font (size 1.27 1.27)) hide)
+    )
+    (property "部品名" "1/4Wカーボン抵抗" (at 193.04 67.31 0)
       (effects (font (size 1.27 1.27)) hide)
     )
@@
     )
     (property "Datasheet" "~" (at 102.87 147.32 0)
+      (effects (font (size 1.27 1.27)) hide)
+    )
+    (property "購入先(参考)" "" (at 102.87 147.32 0)
+      (effects (font (size 1.27 1.27)) hide)
+    )
+    (property "部品名" "1/4Wカーボン抵抗" (at 102.87 147.32 0)
       (effects (font (size 1.27 1.27)) hide)
     )
@@
       (effects (font (size 1.27 1.27)) hide)
     )
+    (property "購入先(参考)" "" (at 193.04 39.37 0)
+      (effects (font (size 1.27 1.27)) hide)
+    )
+    (property "部品名" "1/4Wカーボン抵抗" (at 193.04 39.37 0)
+      (effects (font (size 1.27 1.27)) hide)
+    )
     (pin "1")
     (pin "2")
@@
       (effects (font (size 1.27 1.27)) hide)
     )
-    (property "Datasheet" "http://www.ti.com/lit/gpn/sn74LS125" (at 220.98 107.95 0)
+    (property "Datasheet" "http://www.ti.com/lit/gpn/sn74HC125" (at 220.98 107.95 0)
+      (effects (font (size 1.27 1.27)) hide)
+    )
+    (property "購入先(参考)" "" (at 220.98 107.95 0)
+      (effects (font (size 1.27 1.27)) hide)
+    )
+    (property "部品名" "74HC125" (at 220.98 107.95 0)
       (effects (font (size 1.27 1.27)) hide)
     )
@@
       (effects (font (size 1.27 1.27)) hide)
     )
+    (property "購入先(参考)" "" (at 105.41 147.32 0)
+      (effects (font (size 1.27 1.27)) hide)
+    )
+    (property "部品名" "1/4Wカーボン抵抗" (at 105.41 147.32 0)
+      (effects (font (size 1.27 1.27)) hide)
+    )
     (pin "1")
     (pin "2")
@@
       (effects (font (size 1.27 1.27)) hide)
     )
+    (property "購入先(参考)" "" (at 204.47 53.34 0)
+      (effects (font (size 1.27 1.27)) hide)
+    )
+    (property "部品名" "LED (赤)" (at 204.47 53.34 0)
+      (effects (font (size 1.27 1.27)) hide)
+    )
     (pin "1")
     (pin "2")
@@
     )
     (property "Datasheet" "~" (at 105.41 173.99 0)
+      (effects (font (size 1.27 1.27)) hide)
+    )
+    (property "購入先(参考)" "https://akizukidenshi.com/catalog/g/gP-00586/" (at 105.41 173.99 0)
+      (effects (font (size 1.27 1.27)) hide)
+    )
+    (property "部品名" "4連DIPスイッチ" (at 105.41 173.99 0)
       (effects (font (size 1.27 1.27)) hide)
     )
@@
       (effects (font (size 1.27 1.27)) hide)
     )
+    (property "購入先(参考)" "" (at 204.47 107.95 0)
+      (effects (font (size 1.27 1.27)) hide)
+    )
+    (property "部品名" "LED (黄)" (at 204.47 107.95 0)
+      (effects (font (size 1.27 1.27)) hide)
+    )
     (pin "1")
     (pin "2")
@@
       (effects (font (size 1.27 1.27)) hide)
     )
+    (property "購入先(参考)" "" (at 204.47 67.31 0)
+      (effects (font (size 1.27 1.27)) hide)
+    )
+    (property "部品名" "LED (赤)" (at 204.47 67.31 0)
+      (effects (font (size 1.27 1.27)) hide)
+    )
     (pin "1")
     (pin "2")
@@
       (effects (font (size 1.27 1.27)) hide)
     )
+    (property "購入先(参考)" "" (at 193.04 107.95 0)
+      (effects (font (size 1.27 1.27)) hide)
+    )
+    (property "部品名" "1/4Wカーボン抵抗" (at 193.04 107.95 0)
+      (effects (font (size 1.27 1.27)) hide)
+    )
     (pin "1")
     (pin "2")
@@
     )
     (property "Datasheet" "~" (at 110.49 147.32 0)
+      (effects (font (size 1.27 1.27)) hide)
+    )
+    (property "購入先(参考)" "" (at 110.49 147.32 0)
+      (effects (font (size 1.27 1.27)) hide)
+    )
+    (property "部品名" "1/4Wカーボン抵抗" (at 110.49 147.32 0)
       (effects (font (size 1.27 1.27)) hide)
     )
@@
       (effects (font (size 1.27 1.27)))
     )
-    (property "Value" "AE-CH340E-TYPECH (CH1)" (at 104.775 72.39 0)
+    (property "Value" "AE-CH340E-TYPEC" (at 104.775 72.39 0)
       (effects (font (size 1.27 1.27)))
     )
@@
     )
     (property "Datasheet" "https://akizukidenshi.com/download/ds/akizuki/AE-CH340E-TYPEC.pdf" (at 106.68 68.58 0)
+      (effects (font (size 1.27 1.27)) hide)
+    )
+    (property "購入先(参考)" "https://akizukidenshi.com/catalog/g/gK-14745/" (at 105.41 73.66 0)
+      (effects (font (size 1.27 1.27)) hide)
+    )
+    (property "部品名" "USB-Cシリアル変換モジュール" (at 105.41 73.66 0)
       (effects (font (size 1.27 1.27)) hide)
     )
@@
       (effects (font (size 1.27 1.27)))
     )
-    (property "Value" "AE-CH340E-TYPEC (CH0)" (at 104.775 24.13 0)
+    (property "Value" "AE-CH340E-TYPEC" (at 104.775 24.13 0)
       (effects (font (size 1.27 1.27)))
     )
@@
     )
     (property "Datasheet" "https://akizukidenshi.com/download/ds/akizuki/AE-CH340E-TYPEC.pdf" (at 106.68 20.32 0)
+      (effects (font (size 1.27 1.27)) hide)
+    )
+    (property "購入先(参考)" "https://akizukidenshi.com/catalog/g/gK-14745/" (at 105.41 25.4 0)
+      (effects (font (size 1.27 1.27)) hide)
+    )
+    (property "部品名" "USB-Cシリアル変換モジュール" (at 105.41 25.4 0)
       (effects (font (size 1.27 1.27)) hide)
     )
@@
       (effects (font (size 1.27 1.27)) hide)
     )
+    (property "購入先(参考)" "" (at 107.95 147.32 0)
+      (effects (font (size 1.27 1.27)) hide)
+    )
+    (property "部品名" "1/4Wカーボン抵抗" (at 107.95 147.32 0)
+      (effects (font (size 1.27 1.27)) hide)
+    )
     (pin "1")
     (pin "2")
@@
       (effects (font (size 1.27 1.27)) hide)
     )
-    (property "Datasheet" "https://assets.nexperia.com/documents/data-sheet/74HC_HCT04.pdf" (at 220.98 91.44 0)
+    (property "Datasheet" "http://www.ti.com/lit/gpn/sn74HC04" (at 220.98 91.44 0)
+      (effects (font (size 1.27 1.27)) hide)
+    )
+    (property "購入先(参考)" "" (at 220.98 91.44 0)
+      (effects (font (size 1.27 1.27)) hide)
+    )
+    (property "部品名" "74HC04" (at 220.98 91.44 0)
       (effects (font (size 1.27 1.27)) hide)
     )
@@
       (effects (font (size 1.27 1.27)) hide)
     )
+    (property "購入先(参考)" "" (at 204.47 91.44 0)
+      (effects (font (size 1.27 1.27)) hide)
+    )
+    (property "部品名" "LED (赤)" (at 204.47 91.44 0)
+      (effects (font (size 1.27 1.27)) hide)
+    )
     (pin "1")
     (pin "2")
@@
     )
     (property "Datasheet" "http://www.ti.com/lit/gpn/sn74HC32" (at 220.98 67.31 0)
+      (effects (font (size 1.27 1.27)) hide)
+    )
+    (property "購入先(参考)" "" (at 220.98 67.31 0)
+      (effects (font (size 1.27 1.27)) hide)
+    )
+    (property "部品名" "74HC32" (at 220.98 67.31 0)
       (effects (font (size 1.27 1.27)) hide)
     )
@@
       (effects (font (size 1.27 1.27)) hide)
     )
+    (property "購入先(参考)" "" (at 220.98 53.34 0)
+      (effects (font (size 1.27 1.27)) hide)
+    )
+    (property "部品名" "74HC32" (at 220.98 53.34 0)
+      (effects (font (size 1.27 1.27)) hide)
+    )
     (pin "1")
     (pin "2")
@@
       (effects (font (size 1.27 1.27)) hide)
     )
+    (property "購入先(参考)" "" (at 193.04 91.44 0)
+      (effects (font (size 1.27 1.27)) hide)
+    )
+    (property "部品名" "1/4Wカーボン抵抗" (at 193.04 91.44 0)
+      (effects (font (size 1.27 1.27)) hide)
+    )
     (pin "1")
     (pin "2")
@@
     )
     (property "Datasheet" "~" (at 204.47 39.37 0)
+      (effects (font (size 1.27 1.27)) hide)
+    )
+    (property "購入先(参考)" "" (at 204.47 39.37 0)
+      (effects (font (size 1.27 1.27)) hide)
+    )
+    (property "部品名" "LED (青)" (at 204.47 39.37 0)
       (effects (font (size 1.27 1.27)) hide)
     )
@@
       (effects (font (size 1.27 1.27)) hide)
     )
+    (property "購入先(参考)" "" (at 193.04 53.34 0)
+      (effects (font (size 1.27 1.27)) hide)
+    )
+    (property "部品名" "1/4Wカーボン抵抗" (at 193.04 53.34 0)
+      (effects (font (size 1.27 1.27)) hide)
+    )
     (pin "1")
     (pin "2")
@@
       (effects (font (size 1.27 1.27)) hide)
     )
+    (property "購入先(参考)" "" (at 220.98 39.37 0)
+      (effects (font (size 1.27 1.27)) hide)
+    )
+    (property "部品名" "74HC32" (at 220.98 39.37 0)
+      (effects (font (size 1.27 1.27)) hide)
+    )

Commit message: Update schematics and document.
Parts:
- added R? (x4): 10K, Resistor_THT:R_Axial_DIN0204_L3.6mm_D1.6mm_P7.62mm_Horizontal, symbol Device:R
Connections:
- net LED1: now also R?.2
- net LED2: now also R?.2
- net LED3: now also R?.2
- net VCC: now also R?.1, R?.1, R?.1, R?.1
- net Z80 HALT: now also R?.2
Other:
- moved on the sheet: D?, R?, U?A, U?B, U?C, U?D, U?F
