File: schematics/KiCad/ExtIO_sch.kicad_sch (KiCad schematic)
At the start: 26 parts

Commit message: Update symbol library setting and property value of schematics diagram.
Parts:
- D?: value BUSACK -> /BUSACK
- SW?: value SW_DIP_x04 -> DIP SW
Changed lines of the file:
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@@
       (effects (font (size 1.27 1.27)))
     )
-    (property "Value" "SW_DIP_x04" (at 119.38 172.72 90)
+    (property "Value" "DIP SW" (at 119.38 172.72 90)
       (effects (font (size 1.27 1.27)))
     )
@@
       (effects (font (size 1.27 1.27)))
     )
-    (property "Value" "BUSACK" (at 205.74 113.03 0)
-      (effects (font (size 1.27 1.27)))
-    )
+    (property "Value" "/BUSACK" (at 205.74 113.03 0)
+      (effects (font (size 1.27 1.27)))
+    )

Commit message: Update for MountingHole_Pad.
Parts:
- added REF1, REF2, REF3, REF4: MountingHole_Pad, MountingHole:MountingHole_3.2mm_M3_ISO7380_Pad, symbol Mechanical:MountingHole_Pad
Connections:
- no-connect marks 4 -> 8
Other:
- note added: "Mounting Hole (M3)"
Changed lines of the file:
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@@
   (junction (at 185.42 81.28) (diameter 0) (color 0 0 0 0)
   )
+  (no_connect (at 54.61 168.91))
+  (no_connect (at 54.61 157.48))
   (no_connect (at 110.49 44.45))
+  (no_connect (at 25.4 157.48))
+  (no_connect (at 25.4 168.91))
   (no_connect (at 110.49 77.47))
   (no_connect (at 110.49 92.71))
@@
     (stroke (width 0) (type default))
   )
+  (polyline (pts (xy 78.74 143.51) (xy 78.74 175.26))
+    (stroke (width 0) (type default))
+  )
   (wire (pts (xy 114.3 96.52) (xy 123.19 96.52))
     (stroke (width 0) (type default))
@@
     (stroke (width 0) (type default))
   )
+  (polyline (pts (xy 20.32 143.51) (xy 20.32 175.26))
+    (stroke (width 0) (type default))
+  )
   (wire (pts (xy 238.76 52.07) (xy 242.57 52.07))
     (stroke (width 0) (type default))
@@
     (stroke (width 0) (type default))
   )
+  (polyline (pts (xy 20.32 143.51) (xy 78.74 143.51))
+    (stroke (width 0) (type default))
+  )
   (wire (pts (xy 105.41 157.48) (xy 105.41 166.37))
     (stroke (width 0) (type default))
@@
   )
   (wire (pts (xy 242.57 95.25) (xy 252.73 95.25))
+    (stroke (width 0) (type default))
+  )
+  (polyline (pts (xy 78.74 175.26) (xy 20.32 175.26))
     (stroke (width 0) (type default))
   )
@@
     (fill (type none))
     (effects (font (size 1.27 1.27)) (justify top))
+  )
+  (text "Mounting Hole (M3)" (at 21.59 142.24 0)
+    (effects (font (size 1.27 1.27)) (justify left bottom))
   )
   (hierarchical_label "LED2" (shape input) (at 252.73 81.28 0) (fields_autoplaced)
@@
     )
   )
+  (symbol (lib_id "Mechanical:MountingHole_Pad") (at 54.61 166.37 0) (unit 1)
+    (in_bom yes) (on_board yes) (dnp no) (fields_autoplaced)
+    (property "Reference" "REF4" (at 57.15 163.83 0)
+      (effects (font (size 1.27 1.27)) (justify left))
+    )
+    (property "Value" "MountingHole_Pad" (at 57.15 166.37 0)
+      (effects (font (size 1.27 1.27)) (justify left))
+    )
+    (property "Footprint" "MountingHole:MountingHole_3.2mm_M3_ISO7380_Pad" (at 54.61 166.37 0)
+      (effects (font (size 1.27 1.27)) hide)
+    )
+    (property "Datasheet" "~" (at 54.61 166.37 0)
+      (effects (font (size 1.27 1.27)) hide)
+    )
+    (pin "1")
+    (instances
+      (project "Z80ATmega128"
+        (path "/8c0ff608-9e5b-458c-8fa7-b9973ff97e88/ae537df1-e345-44d5-8641-c1558080fa87"
+          (reference "REF4") (unit 1)
+        )
+      )
+    )
+  )
   (symbol (lib_id "Device:LED") (at 205.74 119.38 180) (unit 1)
     (in_bom yes) (on_board yes) (dnp no)
@@
     )
   )
+  (symbol (lib_id "Mechanical:MountingHole_Pad") (at 25.4 154.94 0) (unit 1)
+    (in_bom yes) (on_board yes) (dnp no) (fields_autoplaced)
+    (property "Reference" "REF1" (at 27.94 152.4 0)
+      (effects (font (size 1.27 1.27)) (justify left))
+    )
+    (property "Value" "MountingHole_Pad" (at 27.94 154.94 0)
+      (effects (font (size 1.27 1.27)) (justify left))
+    )
+    (property "Footprint" "MountingHole:MountingHole_3.2mm_M3_ISO7380_Pad" (at 25.4 154.94 0)
+      (effects (font (size 1.27 1.27)) hide)
+    )
+    (property "Datasheet" "~" (at 25.4 154.94 0)
+      (effects (font (size 1.27 1.27)) hide)
+    )
+    (pin "1")
+    (instances
+      (project "Z80ATmega128"
+        (path "/8c0ff608-9e5b-458c-8fa7-b9973ff97e88/ae537df1-e345-44d5-8641-c1558080fa87"
+          (reference "REF1") (unit 1)
+        )
+      )
+    )
+  )
   (symbol (lib_id "power:GND") (at 222.25 146.05 0) (unit 1)
     (in_bom yes) (on_board yes) (dnp no)
@@
         )
       )
+    )
+  )
+  (symbol (lib_id "Mechanical:MountingHole_Pad") (at 54.61 154.94 0) (unit 1)
+    (in_bom yes) (on_board yes) (dnp no) (fields_autoplaced)
+    (property "Reference" "REF2" (at 57.15 152.4 0)
+      (effects (font (size 1.27 1.27)) (justify left))
+    )
+    (property "Value" "MountingHole_Pad" (at 57.15 154.94 0)
+      (effects (font (size 1.27 1.27)) (justify left))
+    )
+    (property "Footprint" "MountingHole:MountingHole_3.2mm_M3_ISO7380_Pad" (at 54.61 154.94 0)
+      (effects (font (size 1.27 1.27)) hide)
+    )
+    (property "Datasheet" "~" (at 54.61 154.94 0)
+      (effects (font (size 1.27 1.27)) hide)
+    )
+    (pin "1")
+    (instances
+      (project "Z80ATmega128"
+        (path "/8c0ff608-9e5b-458c-8fa7-b9973ff97e88/ae537df1-e345-44d5-8641-c1558080fa87"
+          (reference "REF2") (unit 1)
+        )
+      )
+    )
+  )
+  (symbol (lib_id "Mechanical:MountingHole_Pad") (at 25.4 166.37 0) (unit 1)
+    (in_bom yes) (on_board yes) (dnp no) (fields_autoplaced)
+    (property "Reference" "REF3" (at 27.94 163.83 0)
+      (effects (font (size 1.27 1.27)) (justify left))
+    )
+    (property "Value" "MountingHole_Pad" (at 27.94 166.37 0)
+      (effects (font (size 1.27 1.27)) (justify left))
+    )
+    (property "Footprint" "MountingHole:MountingHole_3.2mm_M3_ISO7380_Pad" (at 25.4 166.37 0)
+      (effects (font (size 1.27 1.27)) hide)
+    )
+    (property "Datasheet" "~" (at 25.4 166.37 0)
+      (effects (font (size 1.27 1.27)) hide)
+    )
+    (pin "1")
+    (instances
+      (project "Z80ATmega128"
+        (path "/8c0ff608-9e5b-458c-8fa7-b9973ff97e88/ae537df1-e345-44d5-8641-c1558080fa87"
+          (reference "REF3") (unit 1)
+        )
+      )

Commit message: Update BOM info and bugfix of PCB2.0
Parts:
- D? (x2): 購入先(参考) (none) -> https://akizukidenshi.com/catalog/g/gI-11639/; 部品名 LED (赤) -> LED (黄)
- D? (x2): 購入先(参考) (none) -> https://akizukidenshi.com/catalog/g/gI-11639/
- D?: 購入先(参考) (none) -> https://akizukidenshi.com/catalog/g/gI-11577/
Changed lines of the file:
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@@
       (effects (font (size 1.27 1.27)) hide)
     )
-    (property "Datasheet" "~" (at 205.74 81.28 0)
-      (effects (font (size 1.27 1.27)) hide)
-    )
-    (property "購入先(参考)" "" (at 205.74 81.28 0)
-      (effects (font (size 1.27 1.27)) hide)
-    )
-    (property "部品名" "LED (赤)" (at 205.74 81.28 0)
+    (property "Datasheet" "https://akizukidenshi.com/download/ds/optosupply/OSR5JA3Z74A.pdf" (at 205.74 81.28 0)
+      (effects (font (size 1.27 1.27)) hide)
+    )
+    (property "購入先(参考)" "https://akizukidenshi.com/catalog/g/gI-11639/" (at 205.74 81.28 0)
+      (effects (font (size 1.27 1.27)) hide)
+    )
+    (property "部品名" "LED (黄)" (at 205.74 81.28 0)
       (effects (font (size 1.27 1.27)) hide)
     )
@@
       (effects (font (size 1.27 1.27)) hide)
     )
-    (property "Datasheet" "~" (at 105.41 173.99 0)
+    (property "Datasheet" "https://akizukidenshi.com/download/ds/excelcell/EDS%20series.pdf" (at 105.41 173.99 0)
       (effects (font (size 1.27 1.27)) hide)
     )
@@
       (effects (font (size 1.27 1.27)) hide)
     )
-    (property "Datasheet" "~" (at 205.74 135.89 0)
-      (effects (font (size 1.27 1.27)) hide)
-    )
-    (property "購入先(参考)" "" (at 205.74 135.89 0)
+    (property "Datasheet" "https://akizukidenshi.com/download/ds/optosupply/OSR5JA3Z74A.pdf" (at 205.74 135.89 0)
+      (effects (font (size 1.27 1.27)) hide)
+    )
+    (property "購入先(参考)" "https://akizukidenshi.com/catalog/g/gI-11639/" (at 205.74 135.89 0)
       (effects (font (size 1.27 1.27)) hide)
     )
@@
       (effects (font (size 1.27 1.27)) hide)
     )
-    (property "Datasheet" "~" (at 205.74 95.25 0)
-      (effects (font (size 1.27 1.27)) hide)
-    )
-    (property "購入先(参考)" "" (at 205.74 95.25 0)
+    (property "Datasheet" "https://akizukidenshi.com/download/ds/optosupply/OSR5JA3Z74A.pdf" (at 205.74 95.25 0)
+      (effects (font (size 1.27 1.27)) hide)
+    )
+    (property "購入先(参考)" "https://akizukidenshi.com/catalog/g/gI-11577/" (at 205.74 95.25 0)
       (effects (font (size 1.27 1.27)) hide)
     )
@@
       (effects (font (size 1.27 1.27)) hide)
     )
-    (property "Datasheet" "~" (at 205.74 119.38 0)
-      (effects (font (size 1.27 1.27)) hide)
-    )
-    (property "購入先(参考)" "" (at 205.74 119.38 0)
-      (effects (font (size 1.27 1.27)) hide)
-    )
-    (property "部品名" "LED (赤)" (at 205.74 119.38 0)
+    (property "Datasheet" "https://akizukidenshi.com/download/ds/optosupply/OSR5JA3Z74A.pdf" (at 205.74 119.38 0)
+      (effects (font (size 1.27 1.27)) hide)
+    )
+    (property "購入先(参考)" "https://akizukidenshi.com/catalog/g/gI-11639/" (at 205.74 119.38 0)
+      (effects (font (size 1.27 1.27)) hide)
+    )
+    (property "部品名" "LED (黄)" (at 205.74 119.38 0)
       (effects (font (size 1.27 1.27)) hide)
     )
@@
       (effects (font (size 1.27 1.27)) hide)
     )
-    (property "Datasheet" "~" (at 205.74 67.31 0)
-      (effects (font (size 1.27 1.27)) hide)
-    )
-    (property "購入先(参考)" "" (at 205.74 67.31 0)
-      (effects (font (size 1.27 1.27)) hide)
-    )
+    (property "Datasheet" "https://akizukidenshi.com/download/ds/optosupply/OSR5JA3Z74A.pdf" (at 205.74 67.31 0)
+      (effects (font (size 1.27 1.27)) hide)
+    )
+    (property "購入先(参考)" "https://akizukidenshi.com/catalog/g/gI-11639/" (at 205.74 67.31 0)
+      (effects (font (size 1.27 1.27)) hide)
+    )
