File: schematics/KiCad/SD_Card.kicad_sch (KiCad schematic)
At the start: 13 parts, among them J6 Micro_SD_Card_Det_Hirose_DM3AT, U14 LP2950-3.3, U16 74HC4050

Commit message: Pull up ISP CLK by 10K ohm resistor.
Parts:
- renumbered R18 to R19, R19 to R20, R20 to R21, R21 to R22, R22 to R23
Changed lines of the file:
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@@
   (title_block
     (title "Micro SD Card interface")
-    (date "2023-08-18")
+    (date "2023-08-27")
     (company "By 46nori")
   )
@@
   (symbol (lib_id "Device:R") (at 90.17 49.53 0) (unit 1)
     (in_bom yes) (on_board yes) (dnp no) (fields_autoplaced)
-    (property "Reference" "R19" (at 92.71 48.2599 0)
+    (property "Reference" "R20" (at 92.71 48.2599 0)
       (effects (font (size 1.27 1.27)) (justify left))
     )
@@
       (project "Z80ATmega128"
         (path "/8c0ff608-9e5b-458c-8fa7-b9973ff97e88/07de70fd-23a2-48ea-a888-9c9311d1e8a8"
-          (reference "R19") (unit 1)
+          (reference "R20") (unit 1)
         )
       )
@@
   (symbol (lib_id "Device:R") (at 157.48 95.25 0) (unit 1)
     (in_bom yes) (on_board yes) (dnp no) (fields_autoplaced)
-    (property "Reference" "R21" (at 160.02 93.9799 0)
+    (property "Reference" "R22" (at 160.02 93.9799 0)
       (effects (font (size 1.27 1.27)) (justify left))
     )
@@
       (project "Z80ATmega128"
         (path "/8c0ff608-9e5b-458c-8fa7-b9973ff97e88/07de70fd-23a2-48ea-a888-9c9311d1e8a8"
-          (reference "R21") (unit 1)
+          (reference "R22") (unit 1)
         )
       )
@@
   (symbol (lib_id "Device:R") (at 146.05 36.83 0) (unit 1)
     (in_bom yes) (on_board yes) (dnp no) (fields_autoplaced)
-    (property "Reference" "R18" (at 148.59 35.5599 0)
+    (property "Reference" "R19" (at 148.59 35.5599 0)
       (effects (font (size 1.27 1.27)) (justify left))
     )
@@
       (project "Z80ATmega128"
         (path "/8c0ff608-9e5b-458c-8fa7-b9973ff97e88/07de70fd-23a2-48ea-a888-9c9311d1e8a8"
-          (reference "R18") (unit 1)
+          (reference "R19") (unit 1)
         )
       )
@@
   (symbol (lib_id "Device:R") (at 125.73 105.41 270) (unit 1)
     (in_bom yes) (on_board yes) (dnp no) (fields_autoplaced)
-    (property "Reference" "R22" (at 125.73 99.06 90)
+    (property "Reference" "R23" (at 125.73 99.06 90)
       (effects (font (size 1.27 1.27)))
     )
@@
       (project "Z80ATmega128"
         (path "/8c0ff608-9e5b-458c-8fa7-b9973ff97e88/07de70fd-23a2-48ea-a888-9c9311d1e8a8"
-          (reference "R22") (unit 1)
+          (reference "R23") (unit 1)
         )
       )
@@
   (symbol (lib_id "Device:R") (at 146.05 69.85 0) (unit 1)
     (in_bom yes) (on_board yes) (dnp no)
-    (property "Reference" "R20" (at 148.59 68.5799 0)
+    (property "Reference" "R21" (at 148.59 68.5799 0)
       (effects (font (size 1.27 1.27)) (justify left))
     )
@@
       (project "Z80ATmega128"
         (path "/8c0ff608-9e5b-458c-8fa7-b9973ff97e88/07de70fd-23a2-48ea-a888-9c9311d1e8a8"
-          (reference "R20") (unit 1)
-        )
-      )
+          (reference "R21") (unit 1)
+        )
+      )

Commit message: Update schematics
Parts:
- removed TP12: 3.3V, TestPoint:TestPoint_Loop_D2.50mm_Drill1.0mm, symbol Connector:TestPoint
- C?: renamed from C12; footprint Capacitor_THT:CP_Radial_Tantal_D5.0mm_P2.50mm -> Capacitor_THT:C_Disc_D3.8mm_W2.6mm_P2.50mm
- C?: renamed from C13; footprint Capacitor_THT:CP_Radial_Tantal_D5.0mm_P2.50mm -> Capacitor_THT:CP_Radial_D5.0mm_P2.50mm
- renumbered C21 to C22, U14 to U?
Connections:
- net VCC: now also R19.2, R20.2; no longer R19.1, R20.1
- net /SD_SS: now also R19.1; no longer R19.2
- net /SD_SW: now also R20.1; no longer R20.2
- net at D2.2 (A): now also R23.1; no longer R23.2
- net at U16.10: now also R23.2; no longer R23.1
Other:
- moved on the sheet: R23

Commit message: Update for PCB design
Parts:
- U?: footprint Package_TO_SOT_THT:TO-92_Inline -> Package_TO_SOT_THT:TO-92_Inline_Wide
Changed lines of the file:
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@@
     (company "By 46nori")
   )
-  (junction (at 49.53 167.64) (diameter 0) (color 0 0 0 0)
+  (junction (at 49.53 168.91) (diameter 0) (color 0 0 0 0)
   )
   (junction (at 107.95 59.69) (diameter 0) (color 0 0 0 0)
@@
     (stroke (width 0) (type default))
   )
+  (wire (pts (xy 63.5 168.91) (xy 63.5 167.64))
+    (stroke (width 0) (type default))
+  )
   (wire (pts (xy 109.22 162.56) (xy 109.22 171.45))
     (stroke (width 0) (type default))
@@
     (stroke (width 0) (type default))
   )
-  (wire (pts (xy 49.53 166.37) (xy 49.53 167.64))
-    (stroke (width 0) (type default))
-  )
-  (wire (pts (xy 49.53 167.64) (xy 63.5 167.64))
+  (wire (pts (xy 49.53 166.37) (xy 49.53 168.91))
+    (stroke (width 0) (type default))
+  )
+  (wire (pts (xy 49.53 168.91) (xy 63.5 168.91))
     (stroke (width 0) (type default))
   )
@@
     (stroke (width 0) (type default))
   )
+  (wire (pts (xy 34.29 168.91) (xy 34.29 167.64))
+    (stroke (width 0) (type default))
+  )
   (wire (pts (xy 129.54 105.41) (xy 130.81 105.41))
     (stroke (width 0) (type default))
@@
     (stroke (width 0) (type default))
   )
-  (wire (pts (xy 49.53 167.64) (xy 49.53 168.91))
+  (wire (pts (xy 49.53 168.91) (xy 49.53 170.18))
     (stroke (width 0) (type default))
   )
@@
     (stroke (width 0) (type default))
   )
-  (wire (pts (xy 34.29 167.64) (xy 49.53 167.64))
+  (wire (pts (xy 34.29 168.91) (xy 49.53 168.91))
     (stroke (width 0) (type default))
   )
@@
       (effects (font (size 1.27 1.27)))
     )
-    (property "Footprint" "Package_TO_SOT_THT:TO-92_Inline" (at 49.53 153.035 0)
+    (property "Footprint" "Package_TO_SOT_THT:TO-92_Inline_Wide" (at 49.53 153.035 0)
       (effects (font (size 1.27 1.27) italic) hide)
     )
@@
     )
   )
-  (symbol (lib_id "power:GND") (at 49.53 168.91 0) (unit 1)
-    (in_bom yes) (on_board yes) (dnp no) (fields_autoplaced)
-    (property "Reference" "#PWR?" (at 49.53 175.26 0)
-      (effects (font (size 1.27 1.27)) hide)
-    )
-    (property "Value" "GND" (at 49.53 173.99 0)
-      (effects (font (size 1.27 1.27)))
-    )
-    (property "Footprint" "" (at 49.53 168.91 0)
-      (effects (font (size 1.27 1.27)) hide)
-    )
-    (property "Datasheet" "" (at 49.53 168.91 0)
-      (effects (font (size 1.27 1.27)) hide)
-    )
+  (symbol (lib_id "power:GND") (at 49.53 170.18 0) (unit 1)
+    (in_bom yes) (on_board yes) (dnp no) (fields_autoplaced)
+    (property "Reference" "#PWR?" (at 49.53 176.53 0)
+      (effects (font (size 1.27 1.27)) hide)
+    )
+    (property "Value" "GND" (at 49.53 175.26 0)
+      (effects (font (size 1.27 1.27)))
+    )
+    (property "Footprint" "" (at 49.53 170.18 0)
+      (effects (font (size 1.27 1.27)) hide)
+    )
+    (property "Datasheet" "" (at 49.53 170.18 0)
+      (effects (font (size 1.27 1.27)) hide)
+    )

Commit message: Update document and BOM of schematics.
Parts:
- C22: 部品名 (none) -> 0.1uF/50V 積層セラミックコンデンサ
- C?: 部品名 (none) -> 1uF/50V 積層セラミックコンデンサ
- C?: 部品名 (none) -> 1uF/50V 電解コンデンサ
- D2: 部品名 (none) -> LED (赤)
- J6: 購入先(参考) (none) -> https://akizukidenshi.com/catalog/g/gC-02395/; 部品名 (none) -> microSDカード用コネクタ
- R19, R20, R21, R22, R23: 部品名 (none) -> 1/4Wカーボン抵抗
- U16: 部品名 (none) -> 74HC4050
- U?: 部品名 (none) -> LP2950-3.3 3.3V三端子レギュレータ
Changed lines of the file:
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@@
+      (effects (font (size 1.27 1.27)) hide)
+    )
+    (property "購入先(参考)" "" (at 49.53 158.75 0)
+      (effects (font (size 1.27 1.27)) hide)
+    )
+    (property "部品名" "LP2950-3.3 3.3V三端子レギュレータ" (at 49.53 158.75 0)
       (effects (font (size 1.27 1.27)) hide)
     )
@@
       (effects (font (size 1.27 1.27)) hide)
     )
-    (property "Datasheet" "http://www.intersil.com/content/dam/intersil/documents/cd40/cd4050bms.pdf" (at 156.21 166.37 0)
+    (property "Datasheet" "https://www.ti.com/lit/ds/symlink/cd74hc4050.pdf" (at 156.21 166.37 0)
+      (effects (font (size 1.27 1.27)) hide)
+    )
+    (property "購入先(参考)" "" (at 156.21 166.37 0)
+      (effects (font (size 1.27 1.27)) hide)
+    )
+    (property "部品名" "74HC4050" (at 156.21 166.37 0)
       (effects (font (size 1.27 1.27)) hide)
     )
@@
       (effects (font (size 1.27 1.27)) hide)
     )
-    (property "Datasheet" "http://www.intersil.com/content/dam/intersil/documents/cd40/cd4050bms.pdf" (at 156.21 152.4 0)
+    (property "Datasheet" "https://www.ti.com/lit/ds/symlink/cd74hc4050.pdf" (at 156.21 152.4 0)
+      (effects (font (size 1.27 1.27)) hide)
+    )
+    (property "購入先(参考)" "" (at 156.21 152.4 0)
+      (effects (font (size 1.27 1.27)) hide)
+    )
+    (property "部品名" "74HC4050" (at 156.21 152.4 0)
       (effects (font (size 1.27 1.27)) hide)
     )
@@
       (effects (font (size 1.27 1.27)) hide)
     )
+    (property "購入先(参考)" "" (at 34.29 163.83 0)
+      (effects (font (size 1.27 1.27)) hide)
+    )
+    (property "部品名" "1uF/50V 積層セラミックコンデンサ" (at 34.29 163.83 0)
+      (effects (font (size 1.27 1.27)) hide)
+    )
     (pin "1")
     (pin "2")
@@
       (effects (font (size 1.27 1.27)) hide)
     )
+    (property "購入先(参考)" "" (at 90.17 49.53 0)
+      (effects (font (size 1.27 1.27)) hide)
+    )
+    (property "部品名" "1/4Wカーボン抵抗" (at 90.17 49.53 0)
+      (effects (font (size 1.27 1.27)) hide)
+    )
     (pin "1")
     (pin "2")
@@
       (effects (font (size 1.27 1.27)) hide)
     )
+    (property "購入先(参考)" "" (at 157.48 95.25 0)
+      (effects (font (size 1.27 1.27)) hide)
+    )
+    (property "部品名" "1/4Wカーボン抵抗" (at 157.48 95.25 0)
+      (effects (font (size 1.27 1.27)) hide)
+    )
     (pin "1")
     (pin "2")
@@
       (effects (font (size 1.27 1.27)) hide)
     )
-    (property "Datasheet" "http://www.intersil.com/content/dam/intersil/documents/cd40/cd4050bms.pdf" (at 124.46 44.45 0)
+    (property "Datasheet" "https://www.ti.com/lit/ds/symlink/cd74hc4050.pdf" (at 124.46 44.45 0)
+      (effects (font (size 1.27 1.27)) hide)
+    )
+    (property "購入先(参考)" "" (at 124.46 44.45 0)
+      (effects (font (size 1.27 1.27)) hide)
+    )
+    (property "部品名" "74HC4050" (at 124.46 44.45 0)
       (effects (font (size 1.27 1.27)) hide)
     )
@@
       (effects (font (size 1.27 1.27)) hide)
     )
+    (property "購入先(参考)" "" (at 118.11 105.41 0)
+      (effects (font (size 1.27 1.27)) hide)
+    )
+    (property "部品名" "LED (赤)" (at 118.11 105.41 0)
+      (effects (font (size 1.27 1.27)) hide)
+    )
     (pin "1")
     (pin "2")
@@
     )
     (property "Datasheet" "https://www.hirose.com/product/en/download_file/key_name/DM3/category/Catalog/doc_file_id/49662/?file_category_id=4&item_id=195&is_series=1" (at 45.72 64.77 0)
+      (effects (font (size 1.27 1.27)) hide)
+    )
+    (property "購入先(参考)" "https://akizukidenshi.com/catalog/g/gC-02395/" (at 45.72 67.31 0)
+      (effects (font (size 1.27 1.27)) hide)
+    )
+    (property "部品名" "microSDカード用コネクタ" (at 45.72 67.31 0)
       (effects (font (size 1.27 1.27)) hide)
     )
@@
       (effects (font (size 1.27 1.27)) hide)
     )
-    (property "Datasheet" "http://www.intersil.com/content/dam/intersil/documents/cd40/cd4050bms.pdf" (at 123.19 158.75 0)
+    (property "Datasheet" "https://www.ti.com/lit/ds/symlink/cd74hc4050.pdf" (at 123.19 158.75 0)
+      (effects (font (size 1.27 1.27)) hide)
+    )
+    (property "購入先(参考)" "" (at 123.19 158.75 0)
+      (effects (font (size 1.27 1.27)) hide)
+    )
+    (property "部品名" "74HC4050" (at 123.19 158.75 0)
       (effects (font (size 1.27 1.27)) hide)
     )
@@
       (effects (font (size 1.27 1.27)) hide)
     )
+    (property "購入先(参考)" "" (at 146.05 36.83 0)
+      (effects (font (size 1.27 1.27)) hide)
+    )
+    (property "部品名" "1/4Wカーボン抵抗" (at 146.05 36.83 0)
+      (effects (font (size 1.27 1.27)) hide)
+    )
     (pin "1")
     (pin "2")
@@
       (effects (font (size 1.27 1.27)) hide)
     )
+    (property "購入先(参考)" "" (at 125.73 105.41 0)
+      (effects (font (size 1.27 1.27)) hide)
+    )
+    (property "部品名" "1/4Wカーボン抵抗" (at 125.73 105.41 0)
+      (effects (font (size 1.27 1.27)) hide)
+    )
     (pin "1")
     (pin "2")
@@
       (effects (font (size 1.27 1.27)) hide)
     )
+    (property "購入先(参考)" "" (at 109.22 158.75 0)
+      (effects (font (size 1.27 1.27)) hide)
+    )
+    (property "部品名" "0.1uF/50V 積層セラミックコンデンサ" (at 109.22 158.75 0)
+      (effects (font (size 1.27 1.27)) hide)
+    )
     (pin "1")
     (pin "2")
@@
     )
     (property "Datasheet" "~" (at 63.5 163.83 0)
+      (effects (font (size 1.27 1.27)) hide)
+    )
+    (property "購入先(参考)" "" (at 63.5 163.83 0)
+      (effects (font (size 1.27 1.27)) hide)
+    )
+    (property "部品名" "1uF/50V 電解コンデンサ" (at 63.5 163.83 0)
       (effects (font (size 1.27 1.27)) hide)
     )
@@
       (effects (font (size 1.27 1.27)) hide)
     )
-    (property "Datasheet" "http://www.intersil.com/content/dam/intersil/documents/cd40/cd4050bms.pdf" (at 124.46 87.63 0)
+    (property "Datasheet" "https://www.ti.com/lit/ds/symlink/cd74hc4050.pdf" (at 124.46 87.63 0)
+      (effects (font (size 1.27 1.27)) hide)
+    )
+    (property "購入先(参考)" "" (at 124.46 87.63 0)
+      (effects (font (size 1.27 1.27)) hide)
+    )
+    (property "部品名" "74HC4050" (at 124.46 87.63 0)
       (effects (font (size 1.27 1.27)) hide)
     )
@@
       (effects (font (size 1.27 1.27)) hide)
     )
+    (property "購入先(参考)" "" (at 146.05 69.85 0)
+      (effects (font (size 1.27 1.27)) hide)
+    )
+    (property "部品名" "1/4Wカーボン抵抗" (at 146.05 69.85 0)
+      (effects (font (size 1.27 1.27)) hide)
+    )
     (pin "1")
     (pin "2")
@@
       (effects (font (size 1.27 1.27)) hide)
     )
-    (property "Datasheet" "http://www.intersil.com/content/dam/intersil/documents/cd40/cd4050bms.pdf" (at 124.46 62.23 0)
+    (property "Datasheet" "https://www.ti.com/lit/ds/symlink/cd74hc4050.pdf" (at 124.46 62.23 0)
+      (effects (font (size 1.27 1.27)) hide)
+    )
+    (property "購入先(参考)" "" (at 124.46 62.23 0)
+      (effects (font (size 1.27 1.27)) hide)
+    )
+    (property "部品名" "74HC4050" (at 124.46 62.23 0)
       (effects (font (size 1.27 1.27)) hide)
     )
@@
       (effects (font (size 1.27 1.27)) hide)
     )
-    (property "Datasheet" "http://www.intersil.com/content/dam/intersil/documents/cd40/cd4050bms.pdf" (at 138.43 105.41 0)
-      (effects (font (size 1.27 1.27)) hide)
-    )
+    (property "Datasheet" "https://www.ti.com/lit/ds/symlink/cd74hc4050.pdf" (at 138.43 105.41 0)
+      (effects (font (size 1.27 1.27)) hide)
+    )
+    (property "購入先(参考)" "" (at 138.43 105.41 0)
+      (effects (font (size 1.27 1.27)) hide)
+    )
+    (property "部品名" "74HC4050" (at 138.43 105.41 0)
+      (effects (font (size 1.27 1.27)) hide)
+    )

Commit message: Update schematics and document.
Parts:
- removed C?: 1u, Capacitor_THT:C_Disc_D3.8mm_W2.6mm_P2.50mm, symbol Device:C
- added C23: 0.1u, Capacitor_THT:C_Disc_D3.8mm_W2.6mm_P2.50mm, symbol Device:C
Connections:
- net GND: now also C23.2
- net VCC: now also C23.1
Changed lines of the file:
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@@
   )
   (symbol (lib_id "Device:C") (at 34.29 163.83 0) (unit 1)
-    (in_bom yes) (on_board yes) (dnp no) (fields_autoplaced)
-    (property "Reference" "C?" (at 38.1 162.5599 0)
+    (in_bom yes) (on_board yes) (dnp no)
+    (property "Reference" "C23" (at 38.1 162.5599 0)
       (effects (font (size 1.27 1.27)) (justify left))
     )
-    (property "Value" "1u" (at 38.1 165.0999 0)
+    (property "Value" "0.1u" (at 38.1 165.0999 0)
       (effects (font (size 1.27 1.27)) (justify left))
     )
@@
       (effects (font (size 1.27 1.27)) hide)
     )
-    (property "部品名" "1uF/50V 積層セラミックコンデンサ" (at 34.29 163.83 0)
+    (property "部品名" "0.1uF/50V 積層セラミックコンデンサ" (at 34.29 163.83 0)
       (effects (font (size 1.27 1.27)) hide)
     )
@@
     (instances
       (project "Z80ATmega128"
-        (path "/8c0ff608-9e5b-458c-8fa7-b9973ff97e88"
-          (reference "C?") (unit 1)
-        )
         (path "/8c0ff608-9e5b-458c-8fa7-b9973ff97e88/07de70fd-23a2-48ea-a888-9c9311d1e8a8"
           (reference "C23") (unit 1)
