File: schematics/KiCad/SD_Card.kicad_sch (KiCad schematic)
At the start: 12 parts, among them J6 Micro_SD_Card_Det_Hirose_DM3AT, U16 74HC4050

Commit message: Update BOM info and bugfix of PCB2.0
Parts:
- D2: 購入先(参考) (none) -> https://akizukidenshi.com/catalog/g/gI-11577/
Changed lines of the file:
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@@
       (effects (font (size 1.27 1.27)) hide)
     )
-    (property "Datasheet" "~" (at 118.11 105.41 0)
+    (property "Datasheet" "https://akizukidenshi.com/download/ds/optosupply/OSR5JA3Z74A.pdf" (at 118.11 105.41 0)
       (effects (font (size 1.27 1.27)) hide)
     )
-    (property "購入先(参考)" "" (at 118.11 105.41 0)
+    (property "購入先(参考)" "https://akizukidenshi.com/catalog/g/gI-11577/" (at 118.11 105.41 0)
       (effects (font (size 1.27 1.27)) hide)
     )
